File: pcb/ai_breakout_LSM9DS0.brd (EAGLE design)
At the start: 15.2 x 19.1 mm, 18 parts, among them J1 1X06, J2 1X06, U1 LSM9DS0

Commit message: minor
Parts:
- U1: device Ai_IC:LGA-24 -> Ai_Sensors:LGA-24
Changed lines of the file:
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@@
 <setting verticaltext="up"/>
 </settings>
-<grid distance="5" unitdist="mil" unit="mil" style="lines" multiple="1" display="yes" altdistance="0.025" altunitdist="inch" altunit="inch"/>
+<grid distance="50" unitdist="mil" unit="mil" style="lines" multiple="1" display="yes" altdistance="0.025" altunitdist="inch" altunit="inch"/>
 <layers>
 <layer number="1" name="Top" color="4" fill="1" visible="yes" active="yes"/>
@@
 </autorouter>
 <elements>
-<element name="U1" library="Ai_IC" package="LGA-24" value="LSM9DS0" x="7.62" y="10.16" smashed="yes" rot="R180">
+<element name="U1" library="Ai_Sensors" package="LGA-24" value="LSM9DS0" x="7.62" y="10.16" smashed="yes" rot="R180">
 <attribute name="NAME" x="10.922" y="7.874" size="0.6096" layer="25" font="vector" ratio="10" rot="R180" align="top-left"/>
 </element>
