File: pcb/ai_breakout_LSM9DS0.brd (EAGLE design)
At the start: 15.2 x 19.1 mm, 18 parts, among them J1 1X06, J2 1X06, U1 LSM9DS0

Commit message: fab done
Parts:
- J2: value 1X06 -> 1X06NOFIRST; device Ai_Connectors:1X06 -> Ai_Connectors:1X06-NOFIRST
- U1: device Ai_IC:LGA-24 -> Ai_Sensors:LGA-24
- turned J1 to 0 degrees
- turned J2 to 180 degrees
Connections:
- net 3V3: now also J1.1; no longer J1.6
- net CS_G: now also J2.5; no longer J2.2
- net CS_XM: now also J2.6; no longer J2.1
- net DRDY_G: now also J2.2; no longer J2.5
- net GND: now also J1.2; no longer J1.5
- net INT1_XM: now also J2.4; no longer J2.3
- net INT2_XM: now also J2.3; no longer J2.4
- net INT_G: now also J2.1; no longer J2.6
- net SCL: now also J1.4; no longer J1.3
- net SDA: now also J1.3; no longer J1.4
- net SDO_G: now also J1.5; no longer J1.2
- net SDO_XM: now also J1.6; no longer J1.1
Routing:
- net CS_XM: track 20.7 -> 22.0 mm
Other:
- outline, holes or cut-outs redrawn
