File: pcb/ai_breakout_LSM9DS0.sch (EAGLE design)
At the start: 18 parts, among them J1 1X06, J2 1X06, U1 LSM9DS0

Commit message: minor
Parts:
- U1: device Ai_IC:LSM9DS0 -> Ai_Sensors:LSM9DS0
Changed lines of the file:
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@@
 </classes>
 <parts>
-<part name="U1" library="Ai_IC" deviceset="LSM9DS0" device=""/>
+<part name="U1" library="Ai_Sensors" deviceset="LSM9DS0" device=""/>
 <part name="U$1" library="Ai_Power" deviceset="3V3" device=""/>
 <part name="GND1" library="Ai_Power" deviceset="GND" device=""/>
