File: pcb/ai_breakout_LSM9DS0.sch (EAGLE design)
At the start: 18 parts, among them J1 1X06, J2 1X06, U1 LSM9DS0

Commit message: fab done
Parts:
- J2: value 1X06 -> 1X06NOFIRST; device Ai_Connectors:1X06 -> Ai_Connectors:1X06NOFIRST
- U1: device Ai_IC:LSM9DS0 -> Ai_Sensors:LSM9DS0
Connections:
- net 3V3: now also J1.1; no longer J1.6
- net CS_G: now also J2.5; no longer J2.2
- net CS_XM: now also J2.6; no longer J2.1
- net DRDY_G: now also J2.2; no longer J2.5
- net GND: now also J1.2; no longer J1.5
- net INT1_XM: now also J2.4; no longer J2.3
- net INT2_XM: now also J2.3; no longer J2.4
- net INT_G: now also J2.1; no longer J2.6
- net SCL: now also J1.4; no longer J1.3
- net SDA: now also J1.3; no longer J1.4
- net SDO_G: now also J1.5; no longer J1.2
- net SDO_XM: now also J1.6; no longer J1.1
Other:
- moved on the sheet: J1, J2
Changed lines of the file:
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@@
 </classes>
 <parts>
-<part name="U1" library="Ai_IC" deviceset="LSM9DS0" device=""/>
+<part name="U1" library="Ai_Sensors" deviceset="LSM9DS0" device=""/>
 <part name="U$1" library="Ai_Power" deviceset="3V3" device=""/>
 <part name="GND1" library="Ai_Power" deviceset="GND" device=""/>
@@
 <part name="JS3" library="Ai_Connectors" deviceset="1X02-SJ-NC" device="T"/>
 <part name="JS4" library="Ai_Connectors" deviceset="1X02-SJ-NC" device="T"/>
-<part name="J1" library="Ai_Connectors" deviceset="1X06" device=""/>
-<part name="J2" library="Ai_Connectors" deviceset="1X06" device=""/>
 <part name="FRAME1" library="Ai_Miscellany" deviceset="FRAME-LETTER" device="">
 <attribute name="AUTHOR" value="A.I. HARDWARE SITH LORDS"/>
@@
 </part>
 <part name="U$4" library="Ai_Miscellany" deviceset="AI-LOGO" device="XS"/>
+<part name="J1" library="Ai_Connectors" deviceset="1X06" device="" value="1X06"/>
+<part name="J2" library="Ai_Connectors" deviceset="1X06" device="NOFIRST" value="1X06NOFIRST"/>
 </parts>
 <sheets>
@@
 <instance part="JS3" gate="G$1" x="165.1" y="149.86" rot="R90"/>
 <instance part="JS4" gate="G$1" x="170.18" y="149.86" rot="R90"/>
-<instance part="J1" gate="M06X1" x="93.98" y="63.5"/>
-<instance part="J2" gate="M06X1" x="152.4" y="60.96" rot="R180"/>
 <instance part="FRAME1" gate="G$1" x="0" y="0"/>
 <instance part="FRAME1" gate="G$2" x="147.32" y="0"/>
 <instance part="U$4" gate="G$1" x="138.43" y="17.78"/>
+<instance part="J1" gate="M06X1" x="99.06" y="63.5"/>
+<instance part="J2" gate="M06X1" x="152.4" y="63.5" rot="MR0"/>
 </instances>
 <busses>
@@
 </segment>
 <segment>
-<pinref part="J1" gate="M06X1" pin="6"/>
-<wire x1="99.06" y1="68.58" x2="101.6" y2="68.58" width="0.1524" layer="91"/>
-<label x="101.6" y="68.58" size="1.27" layer="95" xref="yes"/>
+<wire x1="104.14" y1="55.88" x2="106.68" y2="55.88" width="0.1524" layer="91"/>
+<label x="106.68" y="55.88" size="1.27" layer="95" rot="MR180" xref="yes"/>
+<pinref part="J1" gate="M06X1" pin="1"/>
 </segment>
 </net>
@@
 </segment>
 <segment>
-<pinref part="J1" gate="M06X1" pin="5"/>
-<wire x1="99.06" y1="66.04" x2="101.6" y2="66.04" width="0.1524" layer="91"/>
-<label x="101.6" y="66.04" size="1.27" layer="95" xref="yes"/>
+<wire x1="104.14" y1="58.42" x2="106.68" y2="58.42" width="0.1524" layer="91"/>
+<label x="106.68" y="58.42" size="1.27" layer="95" rot="MR180" xref="yes"/>
+<pinref part="J1" gate="M06X1" pin="2"/>
 </segment>
 </net>
@@
 </segment>
 <segment>
-<pinref part="J1" gate="M06X1" pin="4"/>
-<wire x1="99.06" y1="63.5" x2="101.6" y2="63.5" width="0.1524" layer="91"/>
-<label x="101.6" y="63.5" size="1.27" layer="95" xref="yes"/>
+<wire x1="104.14" y1="60.96" x2="106.68" y2="60.96" width="0.1524" layer="91"/>
+<label x="106.68" y="60.96" size="1.27" layer="95" rot="MR180" xref="yes"/>
+<pinref part="J1" gate="M06X1" pin="3"/>
 </segment>
 </net>
@@
 </segment>
 <segment>
-<pinref part="J1" gate="M06X1" pin="3"/>
-<wire x1="101.6" y1="60.96" x2="99.06" y2="60.96" width="0.1524" layer="91"/>
-<label x="101.6" y="60.96" size="1.27" layer="95" xref="yes"/>
+<wire x1="106.68" y1="63.5" x2="104.14" y2="63.5" width="0.1524" layer="91"/>
+<label x="106.68" y="63.5" size="1.27" layer="95" rot="MR180" xref="yes"/>
+<pinref part="J1" gate="M06X1" pin="4"/>
 </segment>
 </net>
@@
 </segment>
 <segment>
-<pinref part="J1" gate="M06X1" pin="1"/>
-<wire x1="99.06" y1="55.88" x2="101.6" y2="55.88" width="0.1524" layer="91"/>
-<label x="101.6" y="55.88" size="1.27" layer="95" xref="yes"/>
+<wire x1="104.14" y1="68.58" x2="106.68" y2="68.58" width="0.1524" layer="91"/>
+<label x="106.68" y="68.58" size="1.27" layer="95" rot="MR180" xref="yes"/>
+<pinref part="J1" gate="M06X1" pin="6"/>
 </segment>
 </net>
@@
 </segment>
 <segment>
-<pinref part="J2" gate="M06X1" pin="1"/>
 <wire x1="147.32" y1="68.58" x2="144.78" y2="68.58" width="0.1524" layer="91"/>
 <label x="144.78" y="68.58" size="1.27" layer="95" rot="R180" xref="yes"/>
+<pinref part="J2" gate="M06X1" pin="6"/>
 </segment>
 </net>
@@
 </segment>
 <segment>
-<pinref part="J1" gate="M06X1" pin="2"/>
-<wire x1="99.06" y1="58.42" x2="101.6" y2="58.42" width="0.1524" layer="91"/>
-<label x="101.6" y="58.42" size="1.27" layer="95" xref="yes"/>
+<wire x1="104.14" y1="66.04" x2="106.68" y2="66.04" width="0.1524" layer="91"/>
+<label x="106.68" y="66.04" size="1.27" layer="95" rot="MR180" xref="yes"/>
+<pinref part="J1" gate="M06X1" pin="5"/>
 </segment>
 </net>
@@
 </segment>
 <segment>
-<pinref part="J2" gate="M06X1" pin="2"/>
 <wire x1="147.32" y1="66.04" x2="144.78" y2="66.04" width="0.1524" layer="91"/>
 <label x="144.78" y="66.04" size="1.27" layer="95" rot="R180" xref="yes"/>
+<pinref part="J2" gate="M06X1" pin="5"/>
 </segment>
 </net>
@@
 </segment>
 <segment>
-<pinref part="J2" gate="M06X1" pin="5"/>
 <wire x1="147.32" y1="58.42" x2="144.78" y2="58.42" width="0.1524" layer="91"/>
 <label x="144.78" y="58.42" size="1.27" layer="95" rot="R180" xref="yes"/>
+<pinref part="J2" gate="M06X1" pin="2"/>
 </segment>
 </net>
@@
 </segment>
 <segment>
-<pinref part="J2" gate="M06X1" pin="6"/>
 <wire x1="147.32" y1="55.88" x2="144.78" y2="55.88" width="0.1524" layer="91"/>
 <label x="144.78" y="55.88" size="1.27" layer="95" rot="R180" xref="yes"/>
+<pinref part="J2" gate="M06X1" pin="1"/>
 </segment>
 </net>
@@
 </segment>
 <segment>
-<pinref part="J2" gate="M06X1" pin="3"/>
 <wire x1="147.32" y1="63.5" x2="144.78" y2="63.5" width="0.1524" layer="91"/>
 <label x="144.78" y="63.5" size="1.27" layer="95" rot="R180" xref="yes"/>
+<pinref part="J2" gate="M06X1" pin="4"/>
 </segment>
 </net>
@@
 </segment>
 <segment>
-<pinref part="J2" gate="M06X1" pin="4"/>
 <wire x1="147.32" y1="60.96" x2="144.78" y2="60.96" width="0.1524" layer="91"/>
 <label x="144.78" y="60.96" size="1.27" layer="95" rot="R180" xref="yes"/>
+<pinref part="J2" gate="M06X1" pin="3"/>
 </segment>
 </net>
@@
 </sheet>
 </sheets>
+<errors>
+</errors>
 </schematic>
 </drawing>
